File: PD_Decoy.kicad_pcb (KiCad board)
At the start: 2 copper layers, 15.4 x 23.1 mm, 8 parts, among them J1 USB_C_Receptacle_USB2.0, U1 CH224K

Commit message: reroute and widen VBUS track for better current-carrying ability
Routing:
- net /VBUS: track 53.8 -> 49.4 mm, vias 13 -> 14
Changed lines of the file:
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@@
   (segment (start 22.266 28.02334) (end 22.266 27.199) (width 0.35) (layer "F.Cu") (net 4))
   (via (at 18.31 28.823) (size 0.8) (drill 0.4) (layers "F.Cu" "B.Cu") (net 4))
-  (via (at 25.656 14.301) (size 0.8) (drill 0.4) (layers "F.Cu" "B.Cu") (free) (net 4))
-  (via (at 24.132 14.301) (size 0.8) (drill 0.4) (layers "F.Cu" "B.Cu") (free) (net 4))
+  (via (at 25.6 14.2) (size 0.8) (drill 0.4) (layers "F.Cu" "B.Cu") (free) (net 4))
+  (via (at 24.132 14.2) (size 0.8) (drill 0.4) (layers "F.Cu" "B.Cu") (free) (net 4))
   (via (at 24.132 12.65) (size 0.8) (drill 0.4) (layers "F.Cu" "B.Cu") (net 4))
   (via (at 22.354 12.65) (size 0.8) (drill 0.4) (layers "F.Cu" "B.Cu") (free) (net 4))
   (via (at 17.528 25.944) (size 0.8) (drill 0.4) (layers "F.Cu" "B.Cu") (net 4))
+  (via (at 22.4 14.2) (size 0.8) (drill 0.4) (layers "F.Cu" "B.Cu") (free) (net 4))
   (via (at 19.11 28.823) (size 0.8) (drill 0.4) (layers "F.Cu" "B.Cu") (net 4))
   (via (at 19.91 28.823) (size 0.8) (drill 0.4) (layers "F.Cu" "B.Cu") (net 4))
@@
   (via (at 25.656 12.65) (size 0.8) (drill 0.4) (layers "F.Cu" "B.Cu") (free) (net 4))
   (segment (start 18.31 28.823) (end 21.51 28.823) (width 1) (layer "B.Cu") (net 4))
-  (segment (start 17.528 21.159) (end 17.528 25.944) (width 1) (layer "B.Cu") (net 4))
+  (segment (start 20.2 26.054795) (end 17.638795 26.054795) (width 1) (layer "B.Cu") (net 4))
   (segment (start 18.31 26.726) (end 17.638795 26.054795) (width 1) (layer "B.Cu") (net 4))
   (segment (start 17.638795 26.054795) (end 17.528 25.944) (width 1) (layer "B.Cu") (net 4))
-  (segment (start 24.132 14.555) (end 17.528 21.159) (width 1) (layer "B.Cu") (net 4))
-  (segment (start 17.401 21.88) (end 17.401 15.784) (width 0.25) (layer "B.Cu") (net 4))
-  (segment (start 22.2905 26.054795) (end 17.638795 26.054795) (width 1) (layer "B.Cu") (net 4))
+  (segment (start 20.2 26.054795) (end 20.2 16.582) (width 2) (layer "B.Cu") (net 4))
   (segment (start 21.51 26.835295) (end 22.2905 26.054795) (width 1) (layer "B.Cu") (net 4))
-  (segment (start 24.132 12.65) (end 24.132 14.555) (width 1) (layer "B.Cu") (net 4))
+  (segment (start 19.402 15.784) (end 17.401 15.784) (width 0.25) (layer "B.Cu") (net 4))
+  (segment (start 20.2 16.582) (end 19.402 15.784) (width 0.25) (layer "B.Cu") (net 4))
+  (segment (start 22.2905 26.054795) (end 20.2 26.054795) (width 1) (layer "B.Cu") (net 4))
   (segment (start 21.51 28.823) (end 21.51 26.835295) (width 1) (layer "B.Cu") (net 4))
+  (segment (start 20.2 16.582) (end 23.808 12.974) (width 2) (layer "B.Cu") (net 4))
   (segment (start 18.31 28.823) (end 18.31 26.726) (width 1) (layer "B.Cu") (net 4))
   (segment (start 22.481 23.958746) (end 22.481 24.450492) (width 0.25) (layer "F.Cu") (net 5))
